File: Hardware/PCB/Source/openFMS.kicad_sch (KiCad schematic)
At the start: 39 parts, among them U1 STM32F030F4Px, U4 ITR9608-F, X1 8 MHz

Commit message: Add input protection for comparator, spare connector, update crystal load caps
Added Schottky diodes (BAT54CW) and current‑limiting resistors (10 kΩ) to protect MCP6541 comparator inputs from overvoltage/ESD. Introduced a spare connector wired to unused microcontroller GPIOs for future expansion. Updated crystal resonator (DSX321G‑8MHz‑12pF) load capacitors to recommended values (e.g., 15–18 pF) for stable oscillation.
Parts:
- removed C9: 4.7 uF, Capacitor_SMD:C_0603_1608Metric, symbol Device:C
- removed R8: 110, Resistor_SMD:R_0603_1608Metric, symbol Device:R
- added C7: 18 pF, Capacitor_SMD:C_0603_1608Metric, symbol Device:C
- added R11, R4, R5: 10k, Resistor_SMD:R_0603_1608Metric, symbol Device:R
- added VD2: BAT54CW, Package_TO_SOT_SMD_AKL:SOT-323_SC-70, symbol Diode_Schottky_AKL:BAT54CW
- added XP2: Conn_01x04, Connector_JST:JST_EH_B4B-EH-A_1x04_P2.50mm_Vertical, symbol Connector_Generic:Conn_01x04
- C10: value 4.7 uF -> 18 pF
- R9: value 10k -> 110
- X1: footprint Crystal_AKL:Crystal_SMD_5032-4Pin_5.0x3.2mm -> Crystal_AKL:Crystal_SMD_3225-4Pin_3.2x2.5mm; PartNumber X50328MQB4SI -> DSX321G 8MHZ 12PF 20PPM
- XP1: footprint Connector_PinHeader_2.54mm:PinHeader_1x04_P2.54mm_Vertical -> Connector_JST:JST_EH_B4B-EH-A_1x04_P2.50mm_Vertical
- renumbered C7 to C1, C8 to C2, C1 to C4, C6 to C5, C3 to C6, C4 to C8, C5 to C9, DA2 to DA1, DD3 to DD1, DD1 to DD2, R10 to R1, R4 to R10, R5 to R12, R3 to R13, R2 to R14, R1 to R15, R6 to R16, R7 to R17, R11 to R2, R12 to R3, R13 to R6, R14 to R7, R15 to R8, U4 to V1, XP2 to XP3
Connections:
- net +3V3: now also R9.1, R11.2; no longer R9.2, V1.1
- net 2V_REF: now also R5.2, VD2.2 (A1); no longer R3.2, VD1.1 (K)
- net GND: now also V1.2, C7.2, XP2.4 (Pin_4)
- net PHOTO_OUT: now also R11.1; no longer R9.1
- net VCC: now also VD2.3 (K), XP2.1 (Pin_1)
- net at R1.2, R2.1: now also R4.1; no longer DD1.4 (-)
- net at U1.3 (PF1), X1.1: now also C10.1
- net at U1.2 (PF0), X1.3: now also C7.1; no longer C10.1
- net PA4: now reaches U1.10 (PA4)
- net PA4: now also XP2.2 (Pin_2)
- net PA5: now reaches U1.11 (PA5)
- net PA5: now also XP2.3 (Pin_3)
- new net: R3.2, R5.1, VD1.1 (K)
- new net: DD1.4 (-), R4.2, VD2.1 (A2)
- new net: R9.2, V1.1
- no-connect marks 0 -> 3
Other:
- moved on the sheet: R1, R2, R3, VD1

Commit message: Edit PCB
Parts:
- renumbered C7 to C3, C10 to C7
Changed lines of the file:
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@@
 	)
 	(junction
-		(at 106.68 52.07)
-		(diameter 0)
-		(color 0 0 0 0)
-	)
-	(junction
 		(at 311.15 187.96)
 		(diameter 0)
@@
 	)
 	(junction
+		(at 106.68 53.34)
+		(diameter 0)
+		(color 0 0 0 0)
+	)
+	(junction
 		(at 387.35 49.53)
 		(diameter 0)
@@
 	(wire
 		(pts
-			(xy 116.84 53.34) (xy 109.22 53.34)
-		)
-		(stroke
-			(width 0)
-			(type default)
-		)
-	)
-	(wire
-		(pts
 			(xy 125.73 186.69) (xy 125.73 189.23)
 		)
@@
 	(wire
 		(pts
-			(xy 109.22 52.07) (xy 106.68 52.07)
+			(xy 106.68 53.34) (xy 116.84 53.34)
 		)
 		(stroke
@@
 	(wire
 		(pts
-			(xy 106.68 52.07) (xy 106.68 53.34)
-		)
-		(stroke
-			(width 0)
-			(type default)
-		)
-	)
-	(wire
-		(pts
 			(xy 321.31 57.15) (xy 321.31 53.34)
 		)
@@
 	(wire
 		(pts
-			(xy 106.68 48.26) (xy 106.68 52.07)
+			(xy 106.68 48.26) (xy 106.68 53.34)
 		)
 		(stroke
@@
 	(wire
 		(pts
-			(xy 109.22 53.34) (xy 109.22 52.07)
-		)
-		(stroke
-			(width 0)
-			(type default)
-		)
-	)
-	(wire
-		(pts
 			(xy 396.24 161.29) (xy 396.24 168.91)
 		)
@@
 		(dnp no)
 		(fields_autoplaced yes)
-		(property "Reference" "C10"
+		(property "Reference" "C7"
 			(at 327.66 180.3399 0)
 			(show_name no)
@@
 			(project "openFMS"
 				(path "/aaeea2c7-bc98-41b6-aa73-c4db520b2dfb"
-					(reference "C10")
+					(reference "C7")
 					(unit 1)
 				)
@@
 		(dnp no)
 		(fields_autoplaced yes)
-		(property "Reference" "C7"
+		(property "Reference" "C3"
 			(at 304.8 180.3399 0)
 			(show_name no)
@@
 			(project "openFMS"
 				(path "/aaeea2c7-bc98-41b6-aa73-c4db520b2dfb"
-					(reference "C7")
+					(reference "C3")
 					(unit 1)
 				)

Commit message: WIP: PCB component placement draft + FreeCAD 3D models
Finished rough component placement on PCB (routing not started). Added draft FreeCAD models for PCB and filament rod to visualize mechanical compatibility.
Connections:
- net +3V3: now also JP2.1 (A); no longer JP2.2 (B)
- net BOOT: now also JP2.2 (B); no longer JP2.1 (A)
Changed lines of the file:
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@@
 	)
 	(symbol
-		(lib_id "Jumper:SolderJumper_2_Open")
-		(at 281.94 182.88 270)
-		(mirror x)
-		(unit 1)
-		(body_style 1)
-		(exclude_from_sim no)
-		(in_bom no)
-		(on_board yes)
-		(in_pos_files yes)
-		(dnp no)
-		(property "Reference" "JP2"
-			(at 279.4 181.6099 90)
-			(show_name no)
-			(do_not_autoplace no)
-			(effects
-				(font
-					(size 1.27 1.27)
-				)
-				(justify right)
-			)
-		)
-		(property "Value" "SolderJumper_2_Open"
-			(at 279.4 184.1499 90)
-			(hide yes)
-			(show_name no)
-			(do_not_autoplace no)
-			(effects
-				(font
-					(size 1.27 1.27)
-				)
-				(justify right)
-			)
-		)
-		(property "Footprint" "Jumper:SolderJumper-2_P1.3mm_Open_TrianglePad1.0x1.5mm"
-			(at 281.94 182.88 0)
-			(hide yes)
-			(show_name no)
-			(do_not_autoplace no)
-			(effects
-				(font
-					(size 1.27 1.27)
-				)
-			)
-		)
-		(property "Datasheet" ""
-			(at 274.32 182.88 0)
-			(hide yes)
-			(show_name no)
-			(do_not_autoplace no)
-			(effects
-				(font
-					(size 1.27 1.27)
-				)
-			)
-		)
-		(property "Description" "Solder Jumper, 2-pole, open"
-			(at 276.86 182.88 0)
-			(hide yes)
-			(show_name no)
-			(do_not_autoplace no)
-			(effects
-				(font
-					(size 1.27 1.27)
-				)
-			)
-		)
-		(pin "2"
-		)
-		(pin "1"
-		)
-		(instances
-			(project "openFMS"
-				(path "/aaeea2c7-bc98-41b6-aa73-c4db520b2dfb"
-					(reference "JP2")
-					(unit 1)
-				)
-			)
-		)
-	)
-	(symbol
 		(lib_id "Device:R")
 		(at 265.43 180.34 0)
@@
 					(unit 1)
 				)
+			)
+		)
+	)
+	(symbol
+		(lib_id "Jumper:SolderJumper_2_Open")
+		(at 281.94 182.88 90)
+		(mirror x)
+		(unit 1)
+		(body_style 1)
+		(exclude_from_sim no)
+		(in_bom no)
+		(on_board yes)
+		(in_pos_files yes)
+		(dnp no)
+		(property "Reference" "JP2"
+			(at 284.48 184.1501 90)
+			(show_name no)
+			(do_not_autoplace no)
+			(effects
+				(font
+					(size 1.27 1.27)
+				)
+				(justify right)
+			)
+		)
+		(property "Value" "SolderJumper_2_Open"
+			(at 284.48 181.6101 90)
+			(hide yes)
+			(show_name no)
+			(do_not_autoplace no)
+			(effects
+				(font
+					(size 1.27 1.27)
+				)
+				(justify right)
+			)
+		)
+		(property "Footprint" "Jumper:SolderJumper-2_P1.3mm_Open_TrianglePad1.0x1.5mm"
+			(at 281.94 182.88 0)
+			(hide yes)
+			(show_name no)
+			(do_not_autoplace no)
+			(effects
+				(font
+					(size 1.27 1.27)
+				)
+			)
+		)
+		(property "Datasheet" ""
+			(at 289.56 182.88 0)
+			(hide yes)
+			(show_name no)
+			(do_not_autoplace no)
+			(effects
+				(font
+					(size 1.27 1.27)
+				)
+			)
+		)
+		(property "Description" "Solder Jumper, 2-pole, open"
+			(at 287.02 182.88 0)
+			(hide yes)
+			(show_name no)
+			(do_not_autoplace no)
+			(effects
+				(font
+					(size 1.27 1.27)
+				)
+			)
+		)
+		(pin "2"
+		)
+		(pin "1"
+		)
+		(instances
+			(project "openFMS"
+				(path "/aaeea2c7-bc98-41b6-aa73-c4db520b2dfb"
+					(reference "JP2")
+					(unit 1)
+				)

Commit message: WIP: routing
Parts:
- added R10, R8: 10k, Resistor_SMD:R_0603_1608Metric, symbol Device:R
- added VT4, VT6: BSS138L, Package_TO_SOT_SMD_AKL:SOT-23, symbol Transistor_MOSFET_AKL:BSS138L
- renumbered R9 to R11, R10 to R12, R11 to R13, R12 to R14, R13 to R15, R14 to R16, R15 to R17, R16 to R18, R17 to R19, R8 to R9, VT4 to VT5
Connections:
- net GND: now also R10.2, R8.2
- net HALL_OUT: now also U1.8 (PA2); no longer U1.14 (PB1)
- net PA4: now also VT6.1 (G); no longer XP2.2 (Pin_2)
- net VCC: now also VT4.3 (D), VT6.3 (D)
- net PA3: now reaches U1.9 (PA3)
- net PA3: now also VT4.1 (G)
- net PA5: no longer names the net of U1.11 (PA5)
- net PA5: no longer XP2.3 (Pin_3)
- new net PA3_SIG: R8.1, VT4.2 (S), XP2.2 (Pin_2)
- new net PA4_SIG: R10.1, VT6.2 (S), XP2.3 (Pin_3)

Commit message: WIP: routing
Connections:
- net FILAMENT_SIG: now also U1.8 (PA2); no longer U1.7 (PA1)
- net HALL_OUT: now also U1.6 (PA0); no longer U1.8 (PA2)
- net MOTION_SIG: now also U1.7 (PA1); no longer U1.6 (PA0)
Changed lines of the file:
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@@
 	(wire
 		(pts
-			(xy 381 165.1) (xy 370.84 165.1)
+			(xy 384.81 165.1) (xy 370.84 165.1)
 		)
 		(stroke
@@
 		)
 	)
-	(label "FILAMENT_SIG"
-		(at 384.81 162.56 180)
-		(effects
-			(font
-				(size 1.27 1.27)
-			)
-			(justify right bottom)
-		)
-	)
 	(label "SWDIO"
 		(at 314.96 231.14 180)
@@
 	)
 	(label "HALL_OUT"
-		(at 381 165.1 180)
+		(at 384.81 160.02 180)
 		(effects
 			(font
@@
 		)
 	)
+	(label "MOTION_SIG"
+		(at 384.81 162.56 180)
+		(effects
+			(font
+				(size 1.27 1.27)
+			)
+			(justify right bottom)
+		)
+	)
 	(label "SWDIO"
 		(at 382.27 185.42 180)
@@
 		)
 	)
-	(label "MOTION_SIG"
-		(at 384.81 160.02 180)
-		(effects
-			(font
-				(size 1.27 1.27)
-			)
-			(justify right bottom)
-		)
-	)
 	(label "I2C_SDA"
 		(at 382.27 182.88 180)
@@
 		(effects
 			(font
+				(size 1.27 1.27)
+			)
+			(justify right bottom)
+		)
+	)
+	(label "FILAMENT_SIG"
+		(at 384.81 165.1 180)
+		(effects
+			(font

Commit message: WIP: routing and mechanical development
Connections:
- net FILAMENT_SIG: now also U1.7 (PA1); no longer U1.8 (PA2)
- net MOTION_SIG: now also U1.8 (PA2); no longer U1.7 (PA1)
- net PA3: now also U1.10 (PA4); no longer U1.9 (PA3)
- net PA4: now also U1.9 (PA3); no longer U1.10 (PA4)
Changed lines of the file:
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@@
-		)
-	)
-	(label "PA4"
-		(at 382.27 170.18 180)
-		(effects
-			(font
-				(size 1.27 1.27)
-			)
-			(justify right bottom)
 		)
 	)
@@
 		)
 	)
+	(label "PA4"
+		(at 382.27 167.64 180)
+		(effects
+			(font
+				(size 1.27 1.27)
+			)
+			(justify right bottom)
+		)
+	)
 	(label "MOTION_SENS"
 		(at 140.97 189.23 180)
@@
 		)
 	)
-	(label "MOTION_SIG"
-		(at 384.81 162.56 180)
+	(label "PA3"
+		(at 382.27 170.18 180)
 		(effects
 			(font
@@
 		)
 	)
+	(label "FILAMENT_SIG"
+		(at 384.81 162.56 180)
+		(effects
+			(font
+				(size 1.27 1.27)
+			)
+			(justify right bottom)
+		)
+	)
 	(label "PA3_SIG"
 		(at 82.55 31.75 180)
@@
 		)
 	)
-	(label "PA3"
-		(at 382.27 167.64 180)
-		(effects
-			(font
-				(size 1.27 1.27)
-			)
-			(justify right bottom)
-		)
-	)
 	(label "NRST"
 		(at 275.59 186.69 180)
@@
 		)
 	)
-	(label "FILAMENT_SIG"
-		(at 384.81 165.1 180)
-		(effects
-			(font
-				(size 1.27 1.27)
-			)
-			(justify right bottom)
-		)
-	)
 	(label "SWCLK"
 		(at 314.96 233.68 180)
 		(effects
 			(font
+				(size 1.27 1.27)
+			)
+			(justify right bottom)
+		)
+	)
+	(label "MOTION_SIG"
+		(at 384.81 165.1 180)
+		(effects
+			(font
