File: Hardware/PCB/Source/openFMS.kicad_pcb (KiCad board)
At the start: 2 copper layers, 25 x 60 mm, 50 parts, among them U1 STM32F030F4Px, X1 8 MHz

Commit message: WIP: routing
Parts:
- removed DD1: MCP6541T-I-LT, Package_TO_SOT_SMD_AKL:SOT-353_SC-70-5
- removed R1, R2, R3, R4, R5, R6: 10k, Resistor_SMD:R_0603_1608Metric
- removed the REF** at (119.5, 95.4)
- removed the REF** at (138.2, 113.8)
- removed VD1: BZV55B2V0, Diode_SMD:D_MiniMELF
- removed VD2: BAT54CW, Package_TO_SOT_SMD_AKL:SOT-323_SC-70
- removed VT1: BSS138L, Package_TO_SOT_SMD_AKL:SOT-23
- removed VT2: Si2301CDS, Package_TO_SOT_SMD_AKL:SOT-23
- added JP3: SolderJumper_2_Open, Jumper:SolderJumper-2_P1.3mm_Open_TrianglePad1.0x1.5mm, F.Cu at (128.2, 97.6)
- added REF**: MountingHole_3.2mm_M3_DIN965, MountingHole:MountingHole_3.2mm_M3_DIN965, F.Cu at (119.8, 113.8)
- added REF**: MountingHole_3.2mm_M3_DIN965, MountingHole:MountingHole_3.2mm_M3_DIN965, F.Cu at (140.2, 60.2)
- added REF**: MountingHole_3.2mm_M3_DIN965, MountingHole:MountingHole_3.2mm_M3_DIN965, F.Cu at (140.2, 113.8)
- moved R7 30.2 mm to (155.7, 100.8)
- moved R9 30.2 mm to (159.7, 100.8)
- moved VT3 30.2 mm to (155.8, 98.0)
- moved VT5 30.2 mm to (159.8, 98.0)
- moved R10 26.6 mm to (159.7, 106.0)
- moved R8 26.6 mm to (155.7, 106.0)
- moved VT4 26.6 mm to (155.8, 103.3)
- moved VT6 26.6 mm to (159.8, 103.3)
- moved R18 13.6 mm to (132.7, 71.5), turned to 180 degrees
- moved R19 11.7 mm to (132.7, 73.1), turned to 180 degrees
- moved XP1 6.18 mm to (119.5, 99.8)
- moved XP2 6.18 mm to (124.6, 99.8)
- moved V1 4.76 mm to (124.8, 59.3)
- moved C5 4.76 mm to (119.0, 70.6)
- moved DD2 4.76 mm to (124.7, 71.7)
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Connections:
- DA1 pad 3: Net-(DA1-EN) -> VCC
Routing:
- net +3V3: track 56.1 -> 9.46 mm, vias 7 -> 0
- net /MOTION_SIG: track 37.2 -> 8.29 mm
- net /FILAMENT_SIG: track 34.5 -> 8.78 mm
- net /FILAMENT_SENS: track 18.8 -> 0.00 mm
- net /PA3: track 23.3 -> 6.88 mm
- net /MOTION_SENS: track 16.1 -> 0.00 mm
- net /PA4: track 23.8 -> 7.72 mm
- net /2V_REF: track 14.2 -> 0.00 mm
- net /PA4_SIG: track 9.98 -> 0.00 mm
- net Net-(DA1-EN): track 9.76 -> 0.00 mm
- net /PA3_SIG: track 6.18 -> 0.00 mm
- net /I2C_SDA: track 20.8 -> 14.8 mm
- net /I2C_SCL: track 23.4 -> 17.6 mm
- net Net-(R1-Pad2): track 5.82 -> 0.00 mm
- net /PHOTO_OUT: track 36.3 -> 30.8 mm
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- removed copper zone on B.Cu, net +3V3
- removed copper zone on B.Cu, net GND
- removed copper zone on F.Cu, net GND
- removed copper zone on F.Cu, net VCC
Other:
- board size 25 x 60 mm -> 27 x 60 mm
